File: Electrical Testing Suite (Hardware)/Electrical Testing Suite (Hardware).kicad_sch (KiCad schematic)
At the start: 9 parts, among them J1 Conn_01x05_Pin, J2 Conn_01x04_Pin

Commit message: updated kicad
Parts:
- added J10, J11: M12 4Pin A-Code Male (Lighting PWR Verification), symbol Connector:Conn_01x04_Pin
- added J3: 480V 4-pin 7/8 Male PWR Verification, symbol Connector:Conn_01x04_Pin
- added J4, J5, J6: 24V 4-pin M8 Male PWR Verification, symbol Connector:Conn_01x04_Pin
- added J7, J8, J9: 24V 4-pin M8 Male PWR Verification, symbol Connector:Conn_01x05_Pin
- added S10, S4, S5: M8 EC Bulkhead, symbol Connector:Conn_01x01_Socket
- added S11: 120V 3-pin 7/8 Female Input Verification, symbol Connector:Conn_01x03_Pin
- added S12, S13, S14, S7, S8: M12 D-Code Bulkhead, symbol Connector:Conn_01x01_Socket
- added S6, S9: M12 X-Code Bulkhead, symbol Connector:Conn_01x01_Socket
- added SF2: M12 8Pin A-code Male Aux Verification, symbol Connector:Conn_01x08_Pin
- J1: value Conn_01x05_Pin -> 24V 5-pin 7/8 Male PWR Verification
- J2: value Conn_01x04_Pin -> 24V 4-pin M8 Male PWR Verification
- S2: value Conn_01x04_Pin -> 480V 4-pin 7/8 Female Output PWR
- S3: value Conn_01x03_Pin -> 120V 3-pin 7/8 Female Output PWR
- SF1: renamed from SF; value Conn_01x08_Pin -> M12 8Pin A-code Female Aux Verification
Connections:
- net GND: now also J3.4 (Pin_4), J7.3 (Pin_3), J8.3 (Pin_3), J9.3 (Pin_3), S11.3 (Pin_3)
- net SF4: now also SF2.4 (Pin_4); no longer SF1.4 (Pin_4)
- net SF5: now also SF2.5 (Pin_5); no longer SF1.5 (Pin_5)
- net S3 (2)0 renamed S3 (2)
- new net 0V16: J9.1 (Pin_1)
- new net 0V_10: J6.3 (Pin_3)
- new net 0V_11: J6.4 (Pin_4)
- new net 0V_12: J7.1 (Pin_1)
- new net 0V_13: J7.2 (Pin_2)
- new net 0V_14: J8.1 (Pin_1)
- new net 0V_15: J8.2 (Pin_2)
- new net 0V_17: J9.2 (Pin_2)
- new net 0V_18: J10.3 (Pin_3)
- new net 0V_19: J10.4 (Pin_4)
- new net 0V_20: J11.3 (Pin_3)
- new net 0V_21: J11.4 (Pin_4)
- new net 0V_6: J4.3 (Pin_3)
- new net 0V_7: J4.4 (Pin_4)
- new net 0V_8: J5.3 (Pin_3)
- new net 0V_9: J5.4 (Pin_4)
- new net Cam1: S7.1 (Pin_1)
- new net Cam2: S8.1 (Pin_1)
- new net Cam3: S12.1 (Pin_1)
- new net Cam4: S13.1 (Pin_1)
- new net EC LOOP Out: S5.1 (Pin_1)
- new net EC MAIN In: S10.1 (Pin_1)
- new net EC MAIN Out: S4.1 (Pin_1)
- new net Ext Cam1: S14.1 (Pin_1)
- new net J10 (1): J10.1 (Pin_1)
- new net J10 (2): J10.2 (Pin_2)
- new net J11 (1): J11.1 (Pin_1)
- new net J11 (2): J11.2 (Pin_2)
- new net J3 (1): J3.1 (Pin_1)
- new net J3 (2): J3.2 (Pin_2)
- new net J3 (3): J3.3 (Pin_3)
- new net J4 (1): J4.1 (Pin_1)
- new net J4 (2): J4.2 (Pin_2)
- new net J5 (1): J5.1 (Pin_1)
- new net J5 (2): J5.2 (Pin_2)
- new net J6 (1): J6.1 (Pin_1)
- new net J6 (2): J6.2 (Pin_2)
- new net J7 (4): J7.4 (Pin_4)
- new net J7 (5): J7.5 (Pin_5)
- new net J8 (4): J8.4 (Pin_4)
- new net J8 (5): J8.5 (Pin_5)
- new net J9 (4): J9.4 (Pin_4)
- new net J9 (5): J9.5 (Pin_5)
- new net Lan Main In: S6.1 (Pin_1)
- new net Lan Main Out: S9.1 (Pin_1)
- new net S11 (1): S11.1 (Pin_1)
- new net S11 (2): S11.2 (Pin_2)
- no-connect marks 0 -> 12
Other:
- added sheet 120V LED 1 (22NZ09.kicad_sch)
- added sheet AMCAM1 (Amcrest_Camera.kicad_sch)
- added sheet AMCAM2 (Amcrest_Camera.kicad_sch)
- added sheet AMCAM3 (Amcrest_Camera.kicad_sch)
- added sheet AMCAM5 (Amcrest_Camera.kicad_sch)
- added sheet EL1009 (EL1008.kicad_sch)
- added sheet EL1010 (EL1008.kicad_sch)
- added sheet NS 1 (USW-ULTRA-60W.kicad_sch)
- note added: "Need conditions for opening and closing safety contactors two test for 24v outputs. One with safety contactor closed one with it open can likely force it open and closed through ecat chain"
- note added: "Need to figure out process for connecting to external network switch and reading in those cameras, Also need process for verifying external cams by connecting to internal network switch"
- note removed: "120V Output 7/8"
- note removed: "24V Input Verification 7/8"
- note removed: "24V Input Verification M8"
- note removed: "480V Output 7/8"
- moved on the sheet: CB3, F1, J1, J2, S2, S3, SF1
