File: Electrical Testing Suite (Hardware)/Electrical Testing Suite (Hardware).kicad_sch (KiCad schematic)
At the start: 36 parts, among them J1 M12 4Pin A-Code Male (Lightin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, J10 120V 3-pin 7/8 Female Input V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, J2 M12 4Pin A-Code Male (Lightin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, J3 24V 4-pin M8 Male PWR Verific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, J4 24V 4-pin M8 Male PWR Verific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, J5 24V 4-pin M8 Male PWR Verific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, J6 24V 4-pin M8 Male PWR Verific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, J7 24V 5-pin 7/8 Male PWR Verifi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, J8 24V 5-pin 7/8 Male PWR Verifi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, J9 480V 4-pin 7/8 Male PWR Verif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

Commit message: updated schematics
Parts:
- added F2, F3, F4, F5: Fuse, symbol Device:Fuse
- renumbered S1 to J11, S2 to J12, S3 to J13, S4 to J14, S5 to J15, S6 to J16, S7 to J17, S8 to J18, S9 to J19, S10 to J20, S11 to J21, S12 to J22, S13 to J23, S14 to J24, S15 to J25, S16 to J26
Connections:
- net SF1: now reaches SF2.1 (Pin_1)
- net SF2: now reaches SF2.2 (Pin_2)
- net SF6: now reaches SF2.6 (Pin_6)
- net SF8: now reaches SF2.8 (Pin_8)
- net at SF1.1 (Pin_1): now also F2.2
- net at SF1.2 (Pin_2): now also F3.2
- net at SF1.6 (Pin_6): now also F4.2
- net at SF1.8 (Pin_8): now also F5.2
- new net 24V_4: F2.1
- new net 24V_5: F3.1
- new net 24V_6: F4.1
- new net 24V_7: F5.1
- no-connect marks 12 -> 4
Other:
- sheet EL1008 renamed EL1008 (1)
- sheet EL1009 renamed EL1008 (2)
- sheet EL1010 renamed EL1008 (3)
- sheet EL9410 ports: added 1, 2, 3, 4, 5, 6, 7, 8; removed 0V In, 0V Out, 0V Out1, 24V In, 24V Out, 24V Out1, PE, PE1
