File: Electrical Testing Suite (Hardware)/Electrical Testing Suite (Hardware).kicad_sch (KiCad schematic)
At the start: 40 parts, among them J1 M12 4Pin A-Code Male (Lightin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, J10 120V 3-pin 7/8 Female Input V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, J11 M12 D-code EC Bulkhead, J12 M12 D-code EC Bulkhead, J13 M12 D-code EC Bulkhead, J14 M12 D-code EC Bulkhead, J15 M8 EC Bulkhead, J16 M8 EC Bulkhead, J17 M8 EC Bulkhead, J18 M8 EC Bulkhead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

Commit message: updated schematics
Other:
- sheet EL2024 ports: added 0V1, 0V2, 0V3, 0V4; removed 5, 6, 7, 8
Changed lines of the file:
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@@
 	(wire
 		(pts
-			(xy 43.18 331.47) (xy 52.07 331.47)
-		)
-		(stroke
-			(width 0)
-			(type default)
-		)
-	)
-	(wire
-		(pts
 			(xy 43.18 152.4) (xy 45.72 152.4)
 		)
@@
 	(wire
 		(pts
+			(xy 43.18 321.31) (xy 52.07 321.31)
+		)
+		(stroke
+			(width 0)
+			(type default)
+		)
+	)
+	(wire
+		(pts
 			(xy 387.35 410.21) (xy 387.35 424.18)
 		)
@@
 	(wire
 		(pts
-			(xy 43.18 328.93) (xy 52.07 328.93)
-		)
-		(stroke
-			(width 0)
-			(type default)
-		)
-	)
-	(wire
-		(pts
 			(xy 113.03 227.33) (xy 114.3 227.33)
 		)
@@
 	(wire
 		(pts
+			(xy 43.18 331.47) (xy 52.07 331.47)
+		)
+		(stroke
+			(width 0)
+			(type default)
+		)
+	)
+	(wire
+		(pts
 			(xy 365.76 381) (xy 372.11 381)
 		)
@@
 		)
 	)
+	(label "SF7"
+		(at 52.07 321.31 0)
+		(effects
+			(font
+				(size 1.27 1.27)
+			)
+			(justify left bottom)
+		)
+	)
 	(label "EC MAIN In"
 		(at 421.64 407.67 0)
@@
 		)
 	)
-	(label "SF7"
-		(at 52.07 331.47 0)
-		(effects
-			(font
-				(size 1.27 1.27)
-			)
-			(justify left bottom)
-		)
-	)
 	(label "J3 (2)"
 		(at 194.31 375.92 0)
@@
 		)
 	)
-	(label "SF5"
-		(at 52.07 328.93 0)
-		(effects
-			(font
-				(size 1.27 1.27)
-			)
-			(justify left bottom)
-		)
-	)
 	(label "S2 (2)"
 		(at 129.54 156.21 0)
@@
 		)
 	)
+	(label "SF5"
+		(at 52.07 331.47 0)
+		(effects
+			(font
+				(size 1.27 1.27)
+			)
+			(justify left bottom)
+		)
+	)
 	(label "SF8"
 		(at 172.72 411.48 0)
@@
 			)
 		)
-		(pin "8" output
-			(at 43.18 313.69 0)
-			(effects
-				(font
-					(size 1.27 1.27)
-				)
-				(justify right)
-			)
-		)
 		(pin "2" output
 			(at 43.18 328.93 0)
@@
 			)
 		)
-		(pin "5" output
-			(at 43.18 321.31 0)
+		(pin "0V4" input
+			(at 43.18 313.69 0)
 			(effects
 				(font
@@
 			)
 		)
-		(pin "6" output
+		(pin "0V2" input
 			(at 43.18 318.77 0)
 			(effects
@@
 			)
 		)
-		(pin "7" output
+		(pin "0V3" input
 			(at 43.18 316.23 0)
 			(effects
 				(font
+					(size 1.27 1.27)
+				)
+				(justify right)
+			)
+		)
+		(pin "0V1" input
+			(at 43.18 321.31 0)
+			(effects
+				(font
