File: Electrical Testing Suite (Hardware)/EL2024.kicad_sch (KiCad schematic)
At the start: 0 parts

Commit message: big changes to Twincat project
Changed lines of the file:
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@@
-		)
-	)
-	(hierarchical_label "5"
-		(shape output)
-		(at 196.85 105.41 0)
-		(effects
-			(font
-				(size 1.27 1.27)
-			)
-			(justify left)
 		)
 	)
@@
 		)
 	)
-	(hierarchical_label "6"
-		(shape output)
-		(at 196.85 111.76 0)
+	(hierarchical_label "0V4"
+		(shape input)
+		(at 194.31 130.81 0)
 		(effects
 			(font
@@
 		)
 	)
-	(hierarchical_label "7"
-		(shape output)
-		(at 196.85 119.38 0)
+	(hierarchical_label "0V3"
+		(shape input)
+		(at 195.58 121.92 0)
+		(effects
+			(font
+				(size 1.27 1.27)
+			)
+			(justify left)
+		)
+	)
+	(hierarchical_label "0V1"
+		(shape input)
+		(at 195.58 107.95 0)
 		(effects
 			(font
@@
 		)
 	)
-	(hierarchical_label "8"
-		(shape output)
-		(at 196.85 127 0)
+	(hierarchical_label "0V2"
+		(shape input)
+		(at 195.58 114.3 0)
 		(effects
 			(font
